Commit message: moved the castor wheel to make work
the castor wheel was immobile and was making the bot dance

File: macro.xacro (robot description, xacro)
@@ -6,7 +6,7 @@
               <mass value="0.2"/>
               <origin rpy="0 1.5707 1.5707" xyz="0 0 0"/>
-              <inertia ixx="0.000526666666667" ixy="0" ixz="0" iyy="0.000526666666667" iyz="0" izz="0.001"/>
+              <inertia ixx="0.000526666666667" ixy="0" ixz="0" 			       iyy="0.000526666666667" iyz="0" izz="0.001"/>
             </inertial>
-            <collision name="link_right_wheel_collision">
+            <collision name="${name}_collision">
               <origin rpy="0 1.5707 1.5707" xyz="0 0 0"/>
               <geometry>
@@ -32,3 +32,7 @@
       </joint>
     </xacro:macro>
+<xacro:macro name="cylinder_inertia" params="mass r l">
+    <inertia ixx="${mass*(3*r*r+l*l)/12}" ixy = "0" ixz = "0"
+                iyy="${mass*(3*r*r+l*l)/12}" iyz = "0" izz="${mass*(r*r)/2}" />
+</xacro:macro>
 </robot>

File: oa.xacro (robot description, xacro)
@@ -10,9 +10,9 @@
       <mass value="5"/>
       <origin rpy="0 0 0" xyz="0 0 0.1"/>
-      <inertia ixx="0.029625" ixy="0" ixz="0" iyy="0.029625" iyz="0" izz="0.009"/>
+      <xacro:cylinder_inertia mass="5" r="0.15" l="0.06" />
     </inertial>
     <collision name="collision_chassis">
       <geometry>
-        <box size="0.3 0.3 0.07"/>
+        <box size="0.3 0.3 0.06"/>
       </geometry>
     </collision>
@@ -20,5 +20,5 @@
       <origin rpy="0 0 0" xyz="0 0 0"/>
       <geometry>
-        <cylinder length="0.06" radius="0.15"/> <!-- size 0.5 0.3 0.07 -->
+        <cylinder length="0.06" radius="0.15"/>
       </geometry>
       <material name="blue"/>
@@ -26,5 +26,5 @@
     <!-- caster front -->
     <collision name="caster_front_collision">
-      <origin rpy=" 0 0 0" xyz="0.1 0 -0.05"/>
+      <origin rpy=" 0 0 0" xyz="0.35 0 -0.05"/>
       <geometry>
         <sphere radius="0.05"/>
@@ -42,5 +42,5 @@
     </collision>
     <visual name="caster_front_visual">
-      <origin rpy=" 0 0 0" xyz="0.1 0 -0.05"/>
+      <origin rpy=" 0 0 0" xyz="0.2 0 -0.05"/>
       <geometry>
         <sphere radius="0.05"/>
@@ -54,3 +54,29 @@
 	<xacro:joint_wheel name="joint_right_wheel"  child="link_right_wheel"  origin_xyz="-0.05 0.15 0"  />
 	<xacro:joint_wheel name="joint_left_wheel"   child="link_left_wheel"   origin_xyz="-0.05 -0.15 0"  />
+ <!-- adding the sensor-->
+    <link name="sensor_laser">
+    <inertial>
+      <origin xyz="0 0 0" rpy="0 0 0" />
+      <mass value="1" />
+      <xacro:cylinder_inertia mass="1" r="0.03" l="0.02" />
+    </inertial>
+    <visual>
+      <origin xyz="0 0 0" rpy="0 0 0" />
+      <geometry>
+        <cylinder radius="0.03" length="0.02"/>
+      </geometry>
+      <material name="white" />
+    </visual>
+    <collision>
+      <origin xyz="0 0 0" rpy="0 0 0"/>
+      <geometry>
+        <cylinder radius="0.05" length="0.1"/>
+      </geometry>
+    </collision>
+  </link>
+  <joint name="joint_sensor_laser" type="fixed">
+    <origin xyz="0.1 0 0.05" rpy="0 0 0"/>
+    <parent link="link_chassis"/>
+    <child link="sensor_laser"/>
+  </joint>
 </robot>
